Commit message: .

File: src/my_car_ws/urdf/my_car.urdf.xacro (robot description, xacro)
@@ -4,4 +4,4 @@
     <xacro:include filename="my_car_base.urdf.xacro" />
     <xacro:include filename="my_car_base_gazebo.urdf.xacro" />
-    <!-- <xacro:include filename="my_car_lidar.urdf.xacro" />  -->
+    <xacro:include filename="my_car_lidar.urdf.xacro" />
 </robot>

File: src/my_car_ws/urdf/my_car_base.urdf.xacro (robot description, xacro)
@@ -1,127 +1,78 @@
 <?xml version="1.0"?>
-<robot name="my_car">
-  <!-- Base Link -->
-  <link name="base_footprint_link">
-    <visual>
-      <geometry>
-        <box size="0.29 0.26 0.12825"/> <!--0.6 0.4 0.2-->
-      </geometry>
-      <origin xyz="0 0 0.1" rpy="0 0 0"/>
-      <material name="blue"/>
-    </visual>
-    <collision>
-      <geometry>
-        <box size="0.29 0.26 0.12825"/>
-      </geometry>
-      <origin xyz="0 0 0.1" rpy="0 0 0"/>
-    </collision>
-    <inertial>
-      <mass value="5.0"/>
-      <origin xyz="0 0 0.1" rpy="0 0 0"/>
-      <inertia ixx="0.1" ixy="0" ixz="0" iyy="0.1" iyz="0" izz="0.1"/>
-    </inertial>
-  </link>
-  <!-- Left Wheel -->
-  <link name="left_wheel_link">
-    <visual>
-      <geometry>
-        <cylinder radius="0.0425" length="0.05"/>
-      </geometry>
-      <origin xyz="0 0 0" rpy="1.5708 0 0"/>
-      <material name="gray"/>
-    </visual>
-    <collision>
-      <geometry>
-        <cylinder radius="0.0425" length="0.05"/>
-      </geometry>
-      <origin xyz="0 0 0" rpy="1.5708 0 0"/>
-    </collision>
-    <inertial>
-      <mass value="1.0"/>
-      <origin xyz="0 0 0" rpy="0 0 0"/>
-      <inertia ixx="0.01" ixy="0" ixz="0" iyy="0.01" iyz="0" izz="0.01"/>
-    </inertial>
-  </link>
-  <joint name="base_left_wheel_joint" type="continuous">
-    <parent link="base_footprint_link"/>
-    <child link="left_wheel_link"/>
-    <origin xyz="-0.0565 0.13 0.035875" rpy="0 0 0"/> <!-- -0.15 .225 0-->
-    <axis xyz="0 1 0"/>
-  </joint>
-  <!-- Right Wheel -->
-  <link name="right_wheel_link">
-    <visual>
-      <geometry>
-        <cylinder radius="0.0425" length="0.05"/>
-      </geometry>
-      <origin xyz="0 0 0" rpy="1.5708 0 0"/>
-      <material name="gray"/>
-    </visual>
-    <collision>
-      <geometry>
-        <cylinder radius="0.0425" length="0.05"/>
-      </geometry>
-      <origin xyz="0 0 0" rpy="1.5708 0 0"/>
-    </collision>
-    <inertial>
-      <mass value="1.0"/>
-      <origin xyz="0 0 0" rpy="0 0 0"/>
-      <inertia ixx="0.01" ixy="0" ixz="0" iyy="0.01" iyz="0" izz="0.01"/>
-    </inertial>
-  </link>
-  <joint name="base_right_wheel_joint" type="continuous">
-    <parent link="base_footprint_link"/>
-    <child link="right_wheel_link"/>
-    <origin xyz="-0.0565 -0.13 0.035875" rpy="0 0 0"/>
-    <axis xyz="0 1 0"/>
-  </joint>
-  <!-- Left Front Wheel (Fixed) -->
-  <link name="left_front_wheel_link">
-    <visual>
-      <geometry>
-        <cylinder radius="0.0425" length="0.05"/>
-      </geometry>
-      <origin xyz="0 0 0" rpy="1.5708 0 0"/>
-      <material name="gray"/>
-    </visual>
-    <collision>
-      <geometry>
-        <cylinder radius="0.0425" length="0.05"/>
-      </geometry>
-      <origin xyz="0 0 0" rpy="1.5708 0 0"/>
-    </collision>
-  </link>
-  <joint name="base_left_front_wheel_joint" type="fixed">
-    <parent link="base_footprint_link"/>
-    <child link="left_front_wheel_link"/>
-    <origin xyz="0.0565 0.13 0.035875" rpy="0 0 0"/>
-  </joint>
-  <!-- Right Front Wheel (Fixed) -->
-  <link name="right_front_wheel_link">
-    <visual>
-      <geometry>
-        <cylinder radius="0.0425" length="0.05"/>
-      </geometry>
-      <origin xyz="0 0 0" rpy="1.5708 0 0"/>
-      <material name="gray"/>
-    </visual>
-    <collision>
-      <geometry>
-        <cylinder radius="0.0425" length="0.05"/>
-      </geometry>
-      <origin xyz="0 0 0" rpy="1.5708 0 0"/>
-    </collision>
-  </link>
-  <joint name="base_right_front_wheel_joint" type="fixed">
-    <parent link="base_footprint_link"/>
-    <child link="right_front_wheel_link"/>
-    <origin xyz="0.0565 -0.13 0.035875" rpy="0 0 0"/>
-  </joint>
-  <!-- Base Footprint -->
-  <link name="base_link"/>
-  <joint name="base_footprint_base_joint" type="fixed">
-    <parent link="base_link"/>
-    <child link="base_footprint_link"/>
-    <origin xyz="0 0 0.1" rpy="0 0 0"/>
-  </joint>
+<robot xmlns:xacro="http://www.ros.org/wiki/xacro">
+    <xacro:property name="base_length" value="0.6" />
+    <xacro:property name="base_width" value="0.4" />
+    <xacro:property name="base_height" value="0.2" />
+    <xacro:property name="wheel_radius" value="0.1" />
+    <xacro:property name="wheel_length" value="0.05" />
+    <link name = "base_footprint" />
+    <link name = "base_link">
+        <visual>
+            <geometry>
+                <box size = "${base_length} ${base_width} ${base_height}"></box>
+            </geometry>
+            <origin xyz = "0 0 ${base_height / 2.0}" rpy = "0 0 0"></origin>
+            <material name = "blue"/>
+        </visual>
+        <collision>
+            <geometry>
+                <box size = "${base_length} ${base_width} ${base_height}"></box>
+            </geometry>
+            <origin xyz = "0 0 ${base_height / 2.0}" rpy = "0 0 0"></origin>
+        </collision>
+        <xacro:box_inertia m="5.0" l="${3*base_length}" w="${3*base_width}" h="${3*base_height}"
+                           xyz="0 0 ${3*base_height / 2.0}" rpy="0 0 0" />
+    </link>
+    <xacro:macro name="wheel_link" params="prefix">
+        <link name = "${prefix}_wheel_link">
+            <visual>
+                <geometry>
+                    <cylinder radius = "${wheel_radius}" length = "${wheel_length}" />
+                </geometry>
+                <origin xyz = "0 0 0" rpy = "${pi / 2.0} 0 0" />
+                <material name = "grey" />
+            </visual>
+            <collision>
+                <geometry>
+                    <cylinder radius = "${wheel_radius}" length = "${wheel_length}" />
+                </geometry>
+                <origin xyz = "0 0 0" rpy = "${pi / 2.0} 0 0" />
+            </collision>
+            <xacro:cylinder_inertia m ="1.0" r="${3*wheel_radius}" h="${3*wheel_length}" xyz=" 0 0 0"
+                                    rpy="${pi / 2.0} 0 0" />
+        </link>
+    </xacro:macro>
+    <xacro:wheel_link prefix="right"/>
+    <xacro:wheel_link prefix="left"/>
+    <xacro:wheel_link prefix="right_front"/>
+    <xacro:wheel_link prefix="left_front"/>
+    <joint name = "base_footprint_base_joint" type = "fixed">
+        <parent link = "base_footprint" />
+        <child link = "base_link" />
+        <origin xyz = "0 0 0.1" rpy = "0 0 0" />
+    </joint>
+    <joint name = "base_right_wheel_joint" type = "continuous">
+        <parent link = "base_link" />
+        <child link = "right_wheel_link" />
+        <origin xyz = "${-base_length / 4.0} ${-(base_width + wheel_length) / 2.0} 0" rpy = "0 0 0" />
+        <axis xyz = "0 1 0" />
+    </joint>
+    <joint name = "base_left_wheel_joint" type = "continuous">
+        <parent link = "base_link" />
+        <child link = "left_wheel_link" />
+        <origin xyz = "${-base_length / 4.0} ${(base_width + wheel_length) / 2.0} 0" rpy = "0 0 0" />
+        <axis xyz = "0 1 0" />
+    </joint>
+    <joint name = "base_right_front_wheel_joint" type = "continuous">
+        <parent link = "base_link" />
+        <child link = "right_front_wheel_link" />
+        <origin xyz = "${base_length / 4.0} ${-(base_width + wheel_length) / 2.0} 0" rpy = "0 0 0" />
+        <axis xyz = "0 1 0" />
+    </joint>
+    <joint name = "base_left_front_wheel_joint" type = "continuous">
+        <parent link = "base_link" />
+        <child link = "left_front_wheel_link" />
+        <origin xyz = "${base_length / 4.0} ${(base_width + wheel_length) / 2.0} 0" rpy = "0 0 0" />
+        <axis xyz = "0 1 0" />
+    </joint>
 </robot>

File: src/my_car_ws/urdf/my_car_base_gazebo.urdf.xacro (robot description, xacro)
@@ -1,6 +1,5 @@
 <?xml version="1.0"?>
 <robot xmlns:xacro="http://www.ros.org/wiki/xacro">
-    <!-- Material definitions for visual appearance -->
-    <gazebo reference="base_footprint_link">
+    <gazebo reference="base_link">
         <material>Gazebo/Blue</material>
     </gazebo>
@@ -13,19 +12,21 @@
     <gazebo reference="right_front_wheel_link">
         <material>Gazebo/Red</material>
+        <mu1 value="1.0" />
+        <mu2 value="1.0" />
     </gazebo>
     <gazebo reference="left_front_wheel_link">
         <material>Gazebo/Red</material>
+        <mu1 value="1.0" />
+        <mu2 value="1.0" />
+    </gazebo>
+    <gazebo reference="right_wheel_link">
+        <material>Gazebo/Red</material>
+        <mu1 value="1.0" />
+        <mu2 value="1.0" />
     </gazebo>
     <gazebo reference="left_wheel_link">
-        <mu1>0.8</mu1>
-        <mu2>0.8</mu2>
-        <kp>100000.0</kp>
-        <kd>1.0</kd>
-    </gazebo>
-    <gazebo reference="right_wheel_link">
-        <mu1>0.8</mu1>
-        <mu2>0.8</mu2>
-        <kp>100000.0</kp>
-        <kd>1.0</kd>
+        <material>Gazebo/Red</material>
+        <mu1 value="1.0" />
+        <mu2 value="1.0" />
     </gazebo>
     <!-- Differential Drive Plugin for Gazebo Classic -->
@@ -36,9 +37,9 @@
             <left_joint>base_left_wheel_joint</left_joint>
             <!-- Physical parameters -->
-            <wheel_separation>0.26</wheel_separation>
-            <wheel_diameter>0.085</wheel_diameter>
+            <wheel_separation>0.45</wheel_separation>
+            <wheel_diameter>0.2</wheel_diameter>
             <!-- Acceleration and velocity limits -->
-            <max_wheel_acceleration>10.0</max_wheel_acceleration>
-            <max_wheel_torque>10.0</max_wheel_torque>
+            <max_wheel_acceleration>4.0</max_wheel_acceleration>
+            <max_wheel_torque>4.0</max_wheel_torque>
             <!-- ROS topic for velocity commands -->
             <command_topic>cmd_vel</command_topic>
@@ -46,5 +47,5 @@
             <odometry_topic>odom</odometry_topic>
             <odometry_frame>odom</odometry_frame>
-            <robot_base_frame>base_link</robot_base_frame>
+            <robot_base_frame>base_footprint</robot_base_frame>
             <publish_odom>true</publish_odom>
             <publish_odom_tf>true</publish_odom_tf>

File: src/my_car_ws/urdf/my_car_lidar.urdf.xacro (robot description, xacro)
@@ -25,5 +25,5 @@
     </link>
     <joint name="base_lidar_joint" type="fixed">
-        <parent link="base_footprint_link"/>
+        <parent link="base_link"/>
         <child link="lidar_link"/>
         <origin xyz="0.1 0 0.2" rpy="0 0 0"/>

Commit message: pid

File: src/my_car_ws/urdf/my_car.urdf.xacro (robot description, xacro)
@@ -5,3 +5,4 @@
     <xacro:include filename="my_car_base_gazebo.urdf.xacro" />
     <xacro:include filename="my_car_lidar.urdf.xacro" />
+    <!-- <xacro:include filename="ultrasonic.urdf.xacro" />  -->
 </robot>

File: src/my_car_ws/urdf/my_car_base.urdf.xacro (robot description, xacro)
@@ -1,9 +1,9 @@
 <?xml version="1.0"?>
 <robot xmlns:xacro="http://www.ros.org/wiki/xacro">
-    <xacro:property name="base_length" value="0.6" />
-    <xacro:property name="base_width" value="0.4" />
-    <xacro:property name="base_height" value="0.2" />
-    <xacro:property name="wheel_radius" value="0.1" />
-    <xacro:property name="wheel_length" value="0.05" />
+    <xacro:property name="base_length" value="0.29" />
+    <xacro:property name="base_width" value="0.26" /> <!--0.6 0.4 0.2-->
+    <xacro:property name="base_height" value="0.12825" />
+    <xacro:property name="wheel_radius" value="0.0425" />
+    <xacro:property name="wheel_length" value="0.02" />
     <link name = "base_footprint" />
     <link name = "base_link">
@@ -21,6 +21,6 @@
             <origin xyz = "0 0 ${base_height / 2.0}" rpy = "0 0 0"></origin>
         </collision>
-        <xacro:box_inertia m="5.0" l="${3*base_length}" w="${3*base_width}" h="${3*base_height}"
-                           xyz="0 0 ${3*base_height / 2.0}" rpy="0 0 0" />
+        <xacro:box_inertia m="5.0" l="${2.5*base_length}" w="${2.5*base_width}" h="${2.5*base_height}"
+                           xyz="0 0 ${2.5*base_height / 2.0}" rpy="0 0 0" />
     </link>
     <xacro:macro name="wheel_link" params="prefix">
@@ -39,5 +39,5 @@
                 <origin xyz = "0 0 0" rpy = "${pi / 2.0} 0 0" />
             </collision>
-            <xacro:cylinder_inertia m ="1.0" r="${3*wheel_radius}" h="${3*wheel_length}" xyz=" 0 0 0"
+            <xacro:cylinder_inertia m ="1.0" r="${2.5*wheel_radius}" h="${2.5*wheel_length}" xyz=" 0 0 0"
                                     rpy="${pi / 2.0} 0 0" />
         </link>
@@ -55,5 +55,5 @@
         <parent link = "base_link" />
         <child link = "right_wheel_link" />
-        <origin xyz = "${-base_length / 4.0} ${-(base_width + wheel_length) / 2.0} 0" rpy = "0 0 0" />
+        <origin xyz = "${-base_length / 2.0 + 0.0885} ${-(base_width / 2.0)} 0" rpy = "0 0 0" />
         <axis xyz = "0 1 0" />
     </joint>
@@ -61,5 +61,5 @@
         <parent link = "base_link" />
         <child link = "left_wheel_link" />
-        <origin xyz = "${-base_length / 4.0} ${(base_width + wheel_length) / 2.0} 0" rpy = "0 0 0" />
+        <origin xyz = "${-base_length / 2.0 + 0.0885} ${(base_width / 2.0)} 0" rpy = "0 0 0" />
         <axis xyz = "0 1 0" />
     </joint>
@@ -67,5 +67,5 @@
         <parent link = "base_link" />
         <child link = "right_front_wheel_link" />
-        <origin xyz = "${base_length / 4.0} ${-(base_width + wheel_length) / 2.0} 0" rpy = "0 0 0" />
+        <origin xyz = "${base_length / 2.0 - 0.0885} ${-(base_width / 2.0)} 0" rpy = "0 0 0" />
         <axis xyz = "0 1 0" />
     </joint>
@@ -73,5 +73,5 @@
         <parent link = "base_link" />
         <child link = "left_front_wheel_link" />
-        <origin xyz = "${base_length / 4.0} ${(base_width + wheel_length) / 2.0} 0" rpy = "0 0 0" />
+        <origin xyz = "${base_length / 2.0 - 0.0885} ${(base_width / 2.0)} 0" rpy = "0 0 0" />
         <axis xyz = "0 1 0" />
     </joint>

File: src/my_car_ws/urdf/my_car_base_gazebo.urdf.xacro (robot description, xacro)
@@ -12,11 +12,11 @@
     <gazebo reference="right_front_wheel_link">
         <material>Gazebo/Red</material>
-        <mu1 value="1.0" />
-        <mu2 value="1.0" />
+        <mu1 value="0.01" />
+        <mu2 value="0.01" />
     </gazebo>
     <gazebo reference="left_front_wheel_link">
         <material>Gazebo/Red</material>
-        <mu1 value="1.0" />
-        <mu2 value="1.0" />
+        <mu1 value="0.01" />
+        <mu2 value="0.01" />
     </gazebo>
     <gazebo reference="right_wheel_link">
@@ -37,8 +37,8 @@
             <left_joint>base_left_wheel_joint</left_joint>
             <!-- Physical parameters -->
-            <wheel_separation>0.45</wheel_separation>
-            <wheel_diameter>0.2</wheel_diameter>
+            <wheel_separation>0.26</wheel_separation> <!--0.45 0.2-->
+            <wheel_diameter>0.085</wheel_diameter>
             <!-- Acceleration and velocity limits -->
-            <max_wheel_acceleration>4.0</max_wheel_acceleration>
+            <max_wheel_acceleration>2.0</max_wheel_acceleration>
             <max_wheel_torque>4.0</max_wheel_torque>
             <!-- ROS topic for velocity commands -->

File: src/my_car_ws/urdf/my_car_lidar.urdf.xacro (robot description, xacro)
@@ -1,6 +1,6 @@
 <?xml version="1.0"?>
 <robot xmlns:xacro="http://www.ros.org/wiki/xacro">
-    <xacro:property name="lidar_radius" value="0.05" />
-    <xacro:property name="lidar_length" value="0.04" />
+    <xacro:property name="lidar_radius" value="0.038" />
+    <xacro:property name="lidar_length" value="0.0268" />
     <!-- <xacro:property name="lidar_length" value="0.01" />
     <xacro:property name="lidar_width" value="0.1" />
@@ -27,5 +27,5 @@
         <parent link="base_link"/>
         <child link="lidar_link"/>
-        <origin xyz="0.1 0 0.2" rpy="0 0 0"/>
+        <origin xyz="${base_length/2 - 0.11667} 0 ${base_height + 0.5 * lidar_length}" rpy="0 0 0"/>
     </joint>
     <gazebo reference="lidar_link">
